Commit message: chore: Update URDF and world files for improved robot description and simulation

File: src/ROBOTIS-OP3-Common/op3_description/urdf/robotis_op3.visuals.xacro (robot description, xacro)
@@ -1,4 +1,5 @@
 <?xml version="1.0"?>
 <robot xmlns:xacro="http://ros.org/wiki/xacro">
+  <xacro:property name="mesh_prefix" value="file://$(find op3_description)/meshes" />
   <!--
   <xacro:property name="pi" value="3.141592654" />
@@ -8,5 +9,5 @@
     <origin xyz="0 0 0" rpy="0 0 0" />
     <geometry>
-      <mesh filename="package://op3_description/meshes/body.stl"  scale="0.001 0.001 0.001"/>
+      <mesh filename="${mesh_prefix}/body.stl"  scale="0.001 0.001 0.001"/>
     </geometry>
     <material name="Grey">
@@ -18,5 +19,5 @@
     <origin xyz="0 0 0" rpy="0 0 0" />
     <geometry>
-      <mesh filename="package://op3_description/meshes/rl1.stl"  scale="0.001 0.001 0.001"/>
+      <mesh filename="${mesh_prefix}/rl1.stl"  scale="0.001 0.001 0.001"/>
     </geometry>
     <material name="Grey">
@@ -28,5 +29,5 @@
     <origin xyz="0 0 0" rpy="0 0 0" />
     <geometry>
-      <mesh filename="package://op3_description/meshes/rl2.stl"  scale="0.001 0.001 0.001"/>
+      <mesh filename="${mesh_prefix}/rl2.stl"  scale="0.001 0.001 0.001"/>
     </geometry>
     <material name="Grey">
@@ -38,5 +39,5 @@
     <origin xyz="0 0 0" rpy="0 0 0" />
     <geometry>
-      <mesh filename="package://op3_description/meshes/rl3.stl"  scale="0.001 0.001 0.001"/>
+      <mesh filename="${mesh_prefix}/rl3.stl"  scale="0.001 0.001 0.001"/>
     </geometry>
     <material name="Grey">
@@ -48,5 +49,5 @@
     <origin xyz="0 0 0" rpy="0 0 0" />
     <geometry>
-      <mesh filename="package://op3_description/meshes/rl4.stl"  scale="0.001 0.001 0.001"/>
+      <mesh filename="${mesh_prefix}/rl4.stl"  scale="0.001 0.001 0.001"/>
     </geometry>
     <material name="Grey">
@@ -58,5 +59,5 @@
     <origin xyz="0 0 0" rpy="0 0 0" />
     <geometry>
-      <mesh filename="package://op3_description/meshes/rl5.stl"  scale="0.001 0.001 0.001"/>
+      <mesh filename="${mesh_prefix}/rl5.stl"  scale="0.001 0.001 0.001"/>
     </geometry>
     <material name="Grey">
@@ -68,5 +69,5 @@
     <origin xyz="0 0 0" rpy="0 0 0" />
     <geometry>
-      <mesh filename="package://op3_description/meshes/rl6.stl"  scale="0.001 0.001 0.001"/>
+      <mesh filename="${mesh_prefix}/rl6.stl"  scale="0.001 0.001 0.001"/>
     </geometry>
     <material name="Grey">
@@ -78,5 +79,5 @@
     <origin xyz="0 0 0" rpy="0 0 0" />
     <geometry>
-      <mesh filename="package://op3_description/meshes/ll1.stl"  scale="0.001 0.001 0.001"/>
+      <mesh filename="${mesh_prefix}/ll1.stl"  scale="0.001 0.001 0.001"/>
     </geometry>
     <material name="Grey">
@@ -88,5 +89,5 @@
     <origin xyz="0 0 0" rpy="0 0 0" />
     <geometry>
-      <mesh filename="package://op3_description/meshes/ll2.stl"  scale="0.001 0.001 0.001"/>
+      <mesh filename="${mesh_prefix}/ll2.stl"  scale="0.001 0.001 0.001"/>
     </geometry>
     <material name="Grey">
@@ -98,5 +99,5 @@
     <origin xyz="0 0 0" rpy="0 0 0" />
     <geometry>
-      <mesh filename="package://op3_description/meshes/ll3.stl"  scale="0.001 0.001 0.001"/>
+      <mesh filename="${mesh_prefix}/ll3.stl"  scale="0.001 0.001 0.001"/>
     </geometry>
     <material name="Grey">
@@ -108,5 +109,5 @@
     <origin xyz="0 0 0" rpy="0 0 0" />
     <geometry>
-      <mesh filename="package://op3_description/meshes/ll4.stl"  scale="0.001 0.001 0.001"/>
+      <mesh filename="${mesh_prefix}/ll4.stl"  scale="0.001 0.001 0.001"/>
     </geometry>
     <material name="Grey">
@@ -118,5 +119,5 @@
     <origin xyz="0 0 0" rpy="0 0 0" />
     <geometry>
-      <mesh filename="package://op3_description/meshes/ll5.stl"  scale="0.001 0.001 0.001"/>
+      <mesh filename="${mesh_prefix}/ll5.stl"  scale="0.001 0.001 0.001"/>
     </geometry>
     <material name="Grey">
@@ -128,5 +129,5 @@
     <origin xyz="0 0 0" rpy="0 0 0" />
     <geometry>
-      <mesh filename="package://op3_description/meshes/ll6.stl"  scale="0.001 0.001 0.001"/>
+      <mesh filename="${mesh_prefix}/ll6.stl"  scale="0.001 0.001 0.001"/>
     </geometry>
     <material name="Grey">
@@ -138,5 +139,5 @@
     <origin xyz="0 0 0" rpy="0 0 0" />
     <geometry>
-      <mesh filename="package://op3_description/meshes/ra1.stl"  scale="0.001 0.001 0.001"/>
+      <mesh filename="${mesh_prefix}/ra1.stl"  scale="0.001 0.001 0.001"/>
     </geometry>
     <material name="Grey">
@@ -148,5 +149,5 @@
     <origin xyz="0 0 0" rpy="0 0 0" />
     <geometry>
-      <mesh filename="package://op3_description/meshes/ra2.stl"  scale="0.001 0.001 0.001"/>
+      <mesh filename="${mesh_prefix}/ra2.stl"  scale="0.001 0.001 0.001"/>
     </geometry>
     <material name="Grey">
@@ -158,5 +159,5 @@
     <origin xyz="0 0 0" rpy="0 0 0" />
     <geometry>
-      <mesh filename="package://op3_description/meshes/ra3.stl"  scale="0.001 0.001 0.001"/>
+      <mesh filename="${mesh_prefix}/ra3.stl"  scale="0.001 0.001 0.001"/>
     </geometry>
     <material name="Grey">
@@ -168,5 +169,5 @@
     <origin xyz="0 0 0" rpy="0 0 0" />
     <geometry>
-      <mesh filename="package://op3_description/meshes/la1.stl"  scale="0.001 0.001 0.001"/>
+      <mesh filename="${mesh_prefix}/la1.stl"  scale="0.001 0.001 0.001"/>
     </geometry>
     <material name="Grey">
@@ -178,5 +179,5 @@
     <origin xyz="0 0 0" rpy="0 0 0" />
     <geometry>
-      <mesh filename="package://op3_description/meshes/la2.stl"  scale="0.001 0.001 0.001"/>
+      <mesh filename="${mesh_prefix}/la2.stl"  scale="0.001 0.001 0.001"/>
     </geometry>
     <material name="Grey">
@@ -188,5 +189,5 @@
     <origin xyz="0 0 0" rpy="0 0 0" />
     <geometry>
-      <mesh filename="package://op3_description/meshes/la3.stl"  scale="0.001 0.001 0.001"/>
+      <mesh filename="${mesh_prefix}/la3.stl"  scale="0.001 0.001 0.001"/>
     </geometry>
     <material name="Grey">
@@ -198,5 +199,5 @@
     <origin xyz="0 0 0" rpy="0 0 0" />
     <geometry>
-      <mesh filename="package://op3_description/meshes/h1.stl"  scale="0.001 0.001 0.001"/>
+      <mesh filename="${mesh_prefix}/h1.stl"  scale="0.001 0.001 0.001"/>
     </geometry>
     <material name="Grey">
@@ -208,5 +209,5 @@
     <origin xyz="0 0 0" rpy="0 0 0" />
     <geometry>
-      <mesh filename="package://op3_description/meshes/h2.stl"  scale="0.001 0.001 0.001"/>
+      <mesh filename="${mesh_prefix}/h2.stl"  scale="0.001 0.001 0.001"/>
     </geometry>
     <material name="Grey">
